File: KiCad/Stardust/Stardust.kicad_sch (KiCad schematic)
At the start: 42 parts, among them J1 12V DC, J10 12V OUT, J2 RJ12, J3 1x2 Connector, J4 Conn_01x04_Pin, J5 Conn_01x04_Pin, J6 1x3 Header, J7 1x2 Connector, J8 Conn_01x19_Pin, J9 5V IN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

Commit message: updated 3d model. Added new model parts. Updated board and firmware. Everything should be working in this rev
Parts:
- removed C3: 10uF, Capacitor_SMD:C_0603_1608Metric_Pad1.08x0.95mm_HandSolder, symbol Device:C_Small
Connections:
- net ESP32_RST is gone; now on net PEC: U1.2 (VP)
- net AUX3: now also U1.11 (D14); no longer U1.12 (D12)
- net AUX4: now also U1.13 (D13)
- net AUX7: now also U1.30 (D23); no longer J8.18 (Pin_18), U1.29 (D22)
- net AUX8: now also J8.18 (Pin_18), U1.8 (D25); no longer U1.9 (D26)
- net DE+: now also U1.7 (D33); no longer U1.8 (D25)
- net DE-: now also U1.6 (D32); no longer U1.7 (D33)
- net DIR1: now also U1.19 (D2); no longer U1.17 (GND)
- net DIR2: now also U1.9 (D26); no longer U1.10 (D27)
- net EN: now also U1.23 (D5); no longer U1.21 (RX2)
- net GND: now also U1.17 (GND); no longer U1.24 (D18), U1.30 (D23)
- net PEC: no longer U1.3 (VN)
- net RA+: now also U1.5 (D35); no longer U1.6 (D32)
- net RA-: now also U1.4 (D34); no longer U1.5 (D35)
- net RX0: now also U1.28 (TX0); no longer U1.27 (RX0)
- net RX2: now also U1.21 (RX2); no longer U1.19 (D2)
- net SCL: now also U1.29 (D22); no longer U1.28 (TX0)
- net SDA: now also U1.26 (D21); no longer U1.25 (D19)
- net STA: now also U1.12 (D12); no longer U1.13 (D13)
- net STEP1: now also U1.24 (D18); no longer U1.22 (TX2)
- net STEP2: now also U1.10 (D27); no longer U1.11 (D14)
- net TX0: now also U1.27 (RX0); no longer U1.26 (D21)
- net TX2: now also U1.22 (TX2); no longer U1.20 (D4)
- net UART_RX: now also U1.3 (VN); no longer U1.4 (D34)
- net UART_TX: now also U1.20 (D4); no longer U1.18 (D15)
- no-connect marks 15 -> 17
