File: KiCad/Stardust/Stardust.kicad_pcb (KiCad board)
At the start: 2 copper layers, 77 x 77 mm, 43 parts, among them J1 12V DC, J10 12V OUT, J2 RJ12, J3 1x2 Connector, J4 Conn_01x04_Pin, J5 Conn_01x04_Pin, J6 1x3 Header, J7 1x2 Connector, J8 Conn_01x19_Pin, J9 5V IN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

Commit message: updated 3d model. Added new model parts. Updated board and firmware. Everything should be working in this rev
Parts:
- removed C3: 10uF, Capacitor_SMD:C_0603_1608Metric_Pad1.08x0.95mm_HandSolder
- moved C6 15.7 mm to (187.5, 105.0), turned to 0 degrees
Connections:
- J8 pad 18: /AUX7 -> /AUX8
- U1 pad 1: +3.3V -> unconnected-(U1-EN-Pad1)
- U1 pad 10: /DIR2 -> /STEP2
- U1 pad 11: /STEP2 -> /AUX3
- U1 pad 12: /AUX3 -> /STA
- U1 pad 13: /STA -> /AUX4
- U1 pad 15: /AUX4 -> +5V
- U1 pad 16: unconnected-(U1-SD2-Pad16) -> +3.3V
- U1 pad 17: unconnected-(U1-SD3-Pad17) -> GND
- U1 pad 19: +5V -> /DIR1
- U1 pad 2: /ESP32_RST -> /PEC
- U1 pad 20: unconnected-(U1-CLK-Pad20) -> /UART_TX
- U1 pad 21: unconnected-(U1-SD0-Pad21) -> /RX2
- U1 pad 22: unconnected-(U1-SD1-Pad22) -> /TX2
- U1 pad 23: unconnected-(U1-IO15-Pad23) -> /EN
- U1 pad 24: unconnected-(U1-IO2-Pad24) -> /STEP1
- U1 pad 25: /DIR1 -> unconnected-(U1-D19-Pad25)
- U1 pad 26: /UART_TX -> /SDA
- U1 pad 27: /RX2 -> /TX0
- U1 pad 28: /TX2 -> /RX0
- U1 pad 29: /EN -> /SCL
- U1 pad 3: /PEC -> /UART_RX
- U1 pad 30: /STEP1 -> /AUX7
- U1 pad 4: /UART_RX -> /RA-
- U1 pad 5: /RA- -> /RA+
- U1 pad 6: /RA+ -> /DE-
- U1 pad 7: /DE- -> /DE+
- U1 pad 8: /DE+ -> /AUX8
- U1 pad 9: /AUX8 -> /DIR2
Routing:
- net GND: track 109.2 -> 144.7 mm, vias 13 -> 23
- net /AUX8: track 2.67 -> 32.9 mm
- net +3.3V: track 228.3 -> 252.7 mm
- net /AUX7: track 73.7 -> 63.3 mm
- net /DIR2: track 70.9 -> 79.5 mm
- net +5V: track 185.0 -> 193.0 mm
- net /TX2: track 35.6 -> 28.4 mm, vias 4 -> 2
- net /EN: track 36.9 -> 43.0 mm
- net /RX2: track 34.5 -> 28.5 mm, vias 4 -> 2
- net /STEP1: track 36.1 -> 41.2 mm
- net /STEP2: track 74.3 -> 70.1 mm
- net /AUX4: track 38.2 -> 34.4 mm, vias 1 -> 2
- net /DIR1: track 31.5 -> 34.8 mm
- net /RX0: track 48.9 -> 52.1 mm, vias 4 -> 3
- net /UART_RX: track 95.2 -> 98.2 mm
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Other:
- board text added: "AUX8"
